Commit message: fix: add world link to suppress KDL root-link inertia warning
KDL does not support a root link with inertia. Adding a massless world
link and a fixed world_to_base joint makes base_link a child link,
resolving the warning without affecting display or control behavior.

Co-Authored-By: Claude Sonnet 4.6 <noreply@anthropic.com>

File: urdf/minibex.urdf.xacro (robot description, xacro)
@@ -135,5 +135,11 @@
     </joint>
   </xacro:macro>
-  <!-- ============ base_link ============ -->
+  <!-- ============ world / base_link ============ -->
+  <link name="world"/>
+  <joint name="world_to_base" type="fixed">
+    <parent link="world"/>
+    <child link="base_link"/>
+    <origin xyz="0 0 0" rpy="0 0 0"/>
+  </joint>
   <link name="base_link">
     <visual>
