Commit message: feat: add MuJoCo ros2_control support (Stage 5)
UNIFIED_HARDWARE_MUJOCO_IMPROVEMENT_PLAN.md Stage 5: migrate the
quadruped's MuJoCo integration onto ros-controls/mujoco_ros2_control,
matching the dual-arm Stage 3/4 pattern.

- minibex.ros2_control.xacro: add minibex_mujoco_joint_control (position
  command; position/velocity/effort state, since MuJoCo position actuators
  don't support the BXI MIT protocol's velocity/kp/kd/effort command
  interfaces) and minibex_mujoco_ros2_control macros. The latter wires
  odom_free_joint_name/odom_topic so the MJCF's base_joint (free joint)
  pose/velocity publishes as nav_msgs/Odometry, and maps the MJCF's IMU
  sensor triplet to a single ros2_control IMU sensor.
- minibex.urdf.xacro: replace the use_ros2_control bool with a
  hardware_mode arg (none/mock/bxi/mujoco), mirroring
  minibexkai_arm_ros2_ws's post-Gazebo-removal xacro structure.
- test/test_ros2_control_xacro.py: static xacro-expansion regression
  tests for all four hardware_mode values (interfaces, odom/IMU params,
  rejection of an unknown mode or a missing mujoco_model).

Verified: xacro expansion for all 4 modes, and end-to-end in
minibexkai_ros2_ws (see its Stage 5 test report for the runtime
verification this depends on).

Co-Authored-By: Claude Sonnet 5 <noreply@anthropic.com>
Claude-Session: https://claude.ai/code/session_01PR7AcVywuoXbzGtyAFDBbD

File: urdf/minibex.ros2_control.xacro (robot description, xacro)
@@ -3,8 +3,14 @@
   <!--
     Minibex ros2_control 定義。
-    - HWプラグイン: bxi_hardware/BxiSystemInterface
-    - 各関節は フルMIT の command interface（position/velocity/kp/kd/effort）と
+    - mock/bxi: bxi_hardware/BxiSystemInterface（またはmock_components/GenericSystem）。
+      各関節はフルMITのcommand interface（position/velocity/kp/kd/effort）と
       state interface（position/velocity/effort/temperature）を公開する。
-    - per-joint の CANマッピングは config_file(yaml) から注入する。
+      per-jointのCANマッピングはconfig_file(yaml)から注入する（mockでも同じyamlを
+      読み込むが、GenericSystemはCAN通信を行わずcommandをそのままstateへ反映する）。
+    - mujoco: mujoco_ros2_control/MujocoSystemInterface（Stage 5）。MJCFのposition
+      actuatorはkp/kdをMJCF側で固定するため、command interfaceはpositionのみ
+      （双腕Stage 3 ADRと同じ方針）。base_linkを駆動するfree joint（base_joint）の
+      姿勢/速度はodom_free_joint_name経由で/odomへ、IMUはMJCF sensorから
+      ros2_control sensorへ直接マッピングする。
   -->
   <xacro:macro name="minibex_joint_control" params="name">
@@ -21,10 +27,24 @@
     </joint>
   </xacro:macro>
-  <xacro:macro name="minibex_ros2_control" params="config_file spec_dir">
+  <xacro:macro name="minibex_mujoco_joint_control" params="name">
+    <joint name="${name}">
+      <command_interface name="position"/>
+      <state_interface name="position"/>
+      <state_interface name="velocity"/>
+      <state_interface name="effort"/>
+    </joint>
+  </xacro:macro>
+  <xacro:macro name="minibex_standalone_ros2_control"
+               params="hardware_mode config_file spec_dir">
     <ros2_control name="minibex_system" type="system">
       <hardware>
-        <plugin>bxi_hardware/BxiSystemInterface</plugin>
-        <param name="config_file">${config_file}</param>
-        <param name="spec_dir">${spec_dir}</param>
+        <xacro:if value="${hardware_mode == 'mock'}">
+          <plugin>mock_components/GenericSystem</plugin>
+        </xacro:if>
+        <xacro:if value="${hardware_mode == 'bxi'}">
+          <plugin>bxi_hardware/BxiSystemInterface</plugin>
+          <param name="config_file">${config_file}</param>
+          <param name="spec_dir">${spec_dir}</param>
+        </xacro:if>
       </hardware>
       <!-- 関節順序: BL, BR, FL, FR × collar, hip, knee -->
@@ -43,3 +63,44 @@
     </ros2_control>
   </xacro:macro>
+  <xacro:macro name="minibex_mujoco_ros2_control" params="mujoco_model headless sim_speed_factor">
+    <ros2_control name="minibex_system" type="system">
+      <hardware>
+        <plugin>mujoco_ros2_control/MujocoSystemInterface</plugin>
+        <param name="mujoco_model">${mujoco_model}</param>
+        <!-- xacro:property経由だとtrue/falseがPython boolへ変換されるため、この場で直接評価する -->
+        <param name="headless">${'true' if str(headless).lower() == 'true' else 'false'}</param>
+        <param name="sim_speed_factor">${sim_speed_factor}</param>
+        <!-- base_linkを駆動するMJCFのfree joint(base_joint)の姿勢/速度をnav_msgs/Odometryとして公開する -->
+        <param name="odom_free_joint_name">base_joint</param>
+        <param name="odom_topic">/odom</param>
+      </hardware>
+      <xacro:minibex_mujoco_joint_control name="BL_collar_joint"/>
+      <xacro:minibex_mujoco_joint_control name="BL_hip_joint"/>
+      <xacro:minibex_mujoco_joint_control name="BL_knee_joint"/>
+      <xacro:minibex_mujoco_joint_control name="BR_collar_joint"/>
+      <xacro:minibex_mujoco_joint_control name="BR_hip_joint"/>
+      <xacro:minibex_mujoco_joint_control name="BR_knee_joint"/>
+      <xacro:minibex_mujoco_joint_control name="FL_collar_joint"/>
+      <xacro:minibex_mujoco_joint_control name="FL_hip_joint"/>
+      <xacro:minibex_mujoco_joint_control name="FL_knee_joint"/>
+      <xacro:minibex_mujoco_joint_control name="FR_collar_joint"/>
+      <xacro:minibex_mujoco_joint_control name="FR_hip_joint"/>
+      <xacro:minibex_mujoco_joint_control name="FR_knee_joint"/>
+      <!-- MJCFのimu_quat/imu_gyro/imu_accel(scene.xml)を単一IMU sensorへマッピングする -->
+      <sensor name="imu">
+        <param name="mujoco_type">imu</param>
+        <param name="mujoco_sensor_name">imu</param>
+        <state_interface name="orientation.x"/>
+        <state_interface name="orientation.y"/>
+        <state_interface name="orientation.z"/>
+        <state_interface name="orientation.w"/>
+        <state_interface name="angular_velocity.x"/>
+        <state_interface name="angular_velocity.y"/>
+        <state_interface name="angular_velocity.z"/>
+        <state_interface name="linear_acceleration.x"/>
+        <state_interface name="linear_acceleration.y"/>
+        <state_interface name="linear_acceleration.z"/>
+      </sensor>
+    </ros2_control>
+  </xacro:macro>
 </robot>

File: urdf/minibex.urdf.xacro (robot description, xacro)
@@ -13,5 +13,8 @@
   <xacro:arg name="config_file" default=""/>
   <xacro:arg name="spec_dir" default=""/>
-  <xacro:arg name="use_ros2_control" default="true"/>
+  <xacro:arg name="hardware_mode" default="none"/>
+  <xacro:arg name="mujoco_model" default=""/>
+  <xacro:arg name="headless" default="true"/>
+  <xacro:arg name="sim_speed_factor" default="1.0"/>
   <material name="body_color">
     <color rgba="0.75 0.75 0.75 1.0"/>
@@ -183,7 +186,24 @@
     scapula_ixy="-1"  calf_iyz="0.000304"/>
   <!-- ============ ros2_control ============ -->
-  <xacro:if value="$(arg use_ros2_control)">
+  <xacro:if value="${'$(arg hardware_mode)' != 'none'}">
     <xacro:include filename="$(find minibex_description)/urdf/minibex.ros2_control.xacro"/>
-    <xacro:minibex_ros2_control config_file="$(arg config_file)" spec_dir="$(arg spec_dir)"/>
+    <xacro:property name="standalone_mode" value="$(arg hardware_mode)"/>
+    <xacro:unless value="${standalone_mode in ['mock', 'bxi', 'mujoco']}">
+      ${xacro.fatal('hardware_mode must be none, mock, bxi, or mujoco')}
+    </xacro:unless>
+    <xacro:if value="${standalone_mode in ['mock', 'bxi']}">
+      <xacro:minibex_standalone_ros2_control
+        hardware_mode="${standalone_mode}"
+        config_file="$(arg config_file)"
+        spec_dir="$(arg spec_dir)"/>
+    </xacro:if>
+    <xacro:if value="${standalone_mode == 'mujoco'}">
+      <xacro:property name="mujoco_model_value"
+        value="${'$(arg mujoco_model)' if '$(arg mujoco_model)' != '' else xacro.fatal('mujoco_model is required when hardware_mode is mujoco')}"/>
+      <xacro:minibex_mujoco_ros2_control
+        mujoco_model="${mujoco_model_value}"
+        headless="$(arg headless)"
+        sim_speed_factor="$(arg sim_speed_factor)"/>
+    </xacro:if>
   </xacro:if>
 </robot>
